Commit message: Make ur and ignition happy

File: ur_description/urdf/ur.urdf.xacro (robot description, xacro)
@@ -31,3 +31,5 @@
      use_fake_hardware="$(arg use_fake_hardware)"
      fake_sensor_commands="$(arg fake_sensor_commands)" />
+  <!-- Ignition -->
+  <xacro:include filename="ur_ignition_plugins.xacro" />
 </robot>

File: ur_description/urdf/ur_macro.xacro (robot description, xacro)
@@ -102,5 +102,5 @@
         </geometry>
       </collision>
-      <xacro:cylinder_inertial radius="${base_inertia_radius}" length="${base_inertia_length}" mass="${base_mass}">
+      <xacro:cylinder_inertial radius="${base_inertia_radius}" length="${base_inertia_length}" mass="1000">
         <origin xyz="0 0 0" rpy="0 0 0" />
       </xacro:cylinder_inertial>
@@ -247,5 +247,5 @@
          <safety_controller soft_lower_limit="${shoulder_pan_lower_limit + safety_pos_margin}" soft_upper_limit="${shoulder_pan_upper_limit - safety_pos_margin}" k_position="${safety_k_position}" k_velocity="0.0"/>
       </xacro:if>
-      <dynamics damping="0" friction="0"/>
+      <dynamics damping="5" friction="5"/>
     </joint>
     <joint name="${prefix}shoulder_lift_joint" type="revolute">
@@ -259,5 +259,5 @@
          <safety_controller soft_lower_limit="${shoulder_lift_lower_limit + safety_pos_margin}" soft_upper_limit="${shoulder_lift_upper_limit - safety_pos_margin}" k_position="${safety_k_position}" k_velocity="0.0"/>
       </xacro:if>
-      <dynamics damping="0" friction="0"/>
+      <dynamics damping="5" friction="5"/>
     </joint>
     <joint name="${prefix}elbow_joint" type="revolute">
@@ -271,5 +271,5 @@
          <safety_controller soft_lower_limit="${elbow_joint_lower_limit + safety_pos_margin}" soft_upper_limit="${elbow_joint_upper_limit - safety_pos_margin}" k_position="${safety_k_position}" k_velocity="0.0"/>
       </xacro:if>
-      <dynamics damping="0" friction="0"/>
+      <dynamics damping="5" friction="5"/>
     </joint>
     <joint name="${prefix}wrist_1_joint" type="revolute">
@@ -283,5 +283,5 @@
          <safety_controller soft_lower_limit="${wrist_1_lower_limit + safety_pos_margin}" soft_upper_limit="${wrist_1_upper_limit - safety_pos_margin}" k_position="${safety_k_position}" k_velocity="0.0"/>
       </xacro:if>
-      <dynamics damping="0" friction="0"/>
+      <dynamics damping="5" friction="5"/>
     </joint>
     <joint name="${prefix}wrist_2_joint" type="revolute">
@@ -295,5 +295,5 @@
          <safety_controller soft_lower_limit="${wrist_2_lower_limit + safety_pos_margin}" soft_upper_limit="${wrist_2_upper_limit - safety_pos_margin}" k_position="${safety_k_position}" k_velocity="0.0"/>
       </xacro:if>
-      <dynamics damping="0" friction="0"/>
+      <dynamics damping="5" friction="5"/>
     </joint>
     <joint name="${prefix}wrist_3_joint" type="revolute">
@@ -307,5 +307,5 @@
          <safety_controller soft_lower_limit="${wrist_3_lower_limit + safety_pos_margin}" soft_upper_limit="${wrist_3_upper_limit - safety_pos_margin}" k_position="${safety_k_position}" k_velocity="0.0"/>
       </xacro:if>
-      <dynamics damping="0" friction="0"/>
+      <dynamics damping="5" friction="5"/>
     </joint>
     <!-- ROS-Industrial 'base' frame - base_link to UR 'Base' Coordinates transform -->
